File: epic_multi_prog/rev_a/epic_multi_prog_a.sch (EAGLE design)
At the start: 44 parts, among them J1 EPIC-PROG-PORT, J2 MICRO_USB_B_HIROSE_ZX62R-B-5P, J3 MEC1-105-02-XX-XX-D-A, J4 TAG_CONNECT_HEADER_EPIC, J5 MICRO_USB_B_MALE_HIROSE_ZX80-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, U1 FT232RL, U2 MAX1555, U3 MAX1555, U4 MAX1555, U5 MAX1555

Commit message: added opo usb connection
Parts:
- renumbered C18 to C12, S7 to S1
Connections:
- removed net N$13: J5.D-
- removed net N$14: J5.D+
- removed net N$15: J5.ID
- removed net N$17: J5.SHIELD
- net !RST_OPO: now also J5.GND
- net GND: now also J5.SHIELD; no longer J5.GND
- net RX_OPO: now also J5.D+
- net TCK_OPO: now also J5.ID
- net TX_OPO: now also J5.D-
Changed lines of the file:
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@@
 <setting verticaltext="up"/>
 </settings>
-<grid distance="0.1" unitdist="inch" unit="inch" style="lines" multiple="1" display="yes" altdistance="0.01" altunitdist="inch" altunit="inch"/>
+<grid distance="0.1" unitdist="inch" unit="inch" style="lines" multiple="1" display="no" altdistance="0.01" altunitdist="inch" altunit="inch"/>
 <layers>
 <layer number="1" name="Top" color="4" fill="1" visible="no" active="no"/>
@@
 <attribute name="DIGIKEY" value="445-1316-1-ND"/>
 </part>
-<part name="C18" library="SparkFun" deviceset="CAP_POL" device="1206" value="10u">
+<part name="C12" library="SparkFun" deviceset="CAP_POL" device="1206" value="10u">
 <attribute name="DIGIKEY" value="478-1655-1-ND"/>
 </part>
@@
 <part name="S5" library="switches" deviceset="COPAL_CJS-1200TA/SPDT" device=""/>
 <part name="S6" library="switches" deviceset="COPAL_CJS-1200TA/SPDT" device=""/>
-<part name="S7" library="switches" deviceset="TE_SSA12/SPDT" device=""/>
+<part name="S1" library="switches" deviceset="TE_SSA12/SPDT" device=""/>
 <part name="J5" library="connector" deviceset="MICRO_USB_B_MALE_HIROSE_ZX80-B-5S" device="">
 <attribute name="MOUSER" value="798-ZX80-B-5S"/>
@@
 <attribute name="DIGIKEY" x="68.58" y="25.4" size="1.27" layer="96" align="bottom-center" display="off"/>
 </instance>
-<instance part="C18" gate="G$1" x="58.42" y="25.4">
+<instance part="C12" gate="G$1" x="58.42" y="25.4">
 <attribute name="DIGIKEY" x="58.42" y="25.4" size="1.27" layer="96" display="off"/>
 </instance>
@@
 <instance part="S5" gate="G$1" x="175.26" y="33.02"/>
 <instance part="S6" gate="G$1" x="210.82" y="38.1"/>
-<instance part="S7" gate="G$1" x="142.24" y="96.52"/>
+<instance part="S1" gate="G$1" x="142.24" y="96.52"/>
 <instance part="J5" gate="G$1" x="48.26" y="167.64" rot="MR0">
 <attribute name="MOUSER" x="48.26" y="167.64" size="1.27" layer="96" rot="MR0" align="bottom-center" display="off"/>
@@
 <wire x1="45.72" y1="50.8" x2="48.26" y2="50.8" width="0.1524" layer="91"/>
 <wire x1="48.26" y1="50.8" x2="48.26" y2="27.94" width="0.1524" layer="91"/>
-<pinref part="C18" gate="G$1" pin="+"/>
+<pinref part="C12" gate="G$1" pin="+"/>
 <wire x1="58.42" y1="27.94" x2="58.42" y2="50.8" width="0.1524" layer="91"/>
 <wire x1="58.42" y1="50.8" x2="48.26" y2="50.8" width="0.1524" layer="91"/>
@@
 <segment>
 <pinref part="GND5" gate="1" pin="GND"/>
-<pinref part="C18" gate="G$1" pin="-"/>
+<pinref part="C12" gate="G$1" pin="-"/>
 <wire x1="58.42" y1="17.78" x2="58.42" y2="20.32" width="0.1524" layer="91"/>
 </segment>
@@
 </segment>
 <segment>
-<pinref part="J5" gate="G$1" pin="GND"/>
-<wire x1="55.88" y1="162.56" x2="68.58" y2="162.56" width="0.1524" layer="91"/>
-<wire x1="68.58" y1="162.56" x2="68.58" y2="157.48" width="0.1524" layer="91"/>
 <pinref part="GND15" gate="1" pin="GND"/>
+<pinref part="J5" gate="G$1" pin="SHIELD"/>
+<wire x1="68.58" y1="160.02" x2="68.58" y2="157.48" width="0.1524" layer="91"/>
+<wire x1="55.88" y1="160.02" x2="68.58" y2="160.02" width="0.1524" layer="91"/>
+<junction x="68.58" y="160.02"/>
 </segment>
 <segment>
@@
 </segment>
 <segment>
-<pinref part="S7" gate="G$1" pin="A"/>
+<pinref part="S1" gate="G$1" pin="A"/>
 <wire x1="149.86" y1="99.06" x2="152.4" y2="99.06" width="0.1524" layer="91"/>
 <label x="152.4" y="99.06" size="1.27" layer="95" xref="yes"/>
@@
 <wire x1="111.76" y1="99.06" x2="137.16" y2="99.06" width="0.1524" layer="91"/>
 <wire x1="137.16" y1="99.06" x2="137.16" y2="96.52" width="0.1524" layer="91"/>
-<pinref part="S7" gate="G$1" pin="IN"/>
+<pinref part="S1" gate="G$1" pin="IN"/>
 <wire x1="137.16" y1="96.52" x2="139.7" y2="96.52" width="0.1524" layer="91"/>
 </segment>
@@
 <junction x="190.5" y="96.52"/>
 </segment>
+<segment>
+<pinref part="J5" gate="G$1" pin="D-"/>
+<wire x1="55.88" y1="170.18" x2="58.42" y2="170.18" width="0.1524" layer="91"/>
+<label x="58.42" y="170.18" size="1.27" layer="95" xref="yes"/>
+</segment>
 </net>
 <net name="RX_OPO" class="0">
@@
 <junction x="190.5" y="109.22"/>
 </segment>
+<segment>
+<pinref part="J5" gate="G$1" pin="D+"/>
+<wire x1="55.88" y1="167.64" x2="58.42" y2="167.64" width="0.1524" layer="91"/>
+<label x="58.42" y="167.64" size="1.27" layer="95" xref="yes"/>
+</segment>
 </net>
 <net name="RX_POGO" class="0">
@@
 <junction x="190.5" y="71.12"/>
 </segment>
+<segment>
+<pinref part="J5" gate="G$1" pin="GND"/>
+<wire x1="55.88" y1="162.56" x2="58.42" y2="162.56" width="0.1524" layer="91"/>
+<label x="58.42" y="162.56" size="1.27" layer="95" xref="yes"/>
+</segment>
 </net>
 <net name="TCK_EDGE" class="0">
@@
 <junction x="190.5" y="83.82"/>
 </segment>
+<segment>
+<pinref part="J5" gate="G$1" pin="ID"/>
+<wire x1="55.88" y1="165.1" x2="58.42" y2="165.1" width="0.1524" layer="91"/>
+<label x="58.42" y="165.1" size="1.27" layer="95" xref="yes"/>
+</segment>
 </net>
 <net name="!RST_EDGE" class="0">
@@
 </segment>
 </net>
-<net name="N$13" class="0">
-<segment>
-<pinref part="J5" gate="G$1" pin="D-"/>
-<wire x1="55.88" y1="170.18" x2="58.42" y2="170.18" width="0.1524" layer="91"/>
-<label x="58.42" y="170.18" size="1.27" layer="95" xref="yes"/>
-</segment>
-</net>
-<net name="N$14" class="0">
-<segment>
-<pinref part="J5" gate="G$1" pin="D+"/>
-<wire x1="55.88" y1="167.64" x2="58.42" y2="167.64" width="0.1524" layer="91"/>
-<label x="58.42" y="167.64" size="1.27" layer="95" xref="yes"/>
-</segment>
-</net>
-<net name="N$15" class="0">
-<segment>
-<pinref part="J5" gate="G$1" pin="ID"/>
-<wire x1="55.88" y1="165.1" x2="58.42" y2="165.1" width="0.1524" layer="91"/>
-<label x="58.42" y="165.1" size="1.27" layer="95" xref="yes"/>
-</segment>
-</net>
-<net name="N$17" class="0">
-<segment>
-<pinref part="J5" gate="G$1" pin="SHIELD"/>
-<wire x1="55.88" y1="160.02" x2="58.42" y2="160.02" width="0.1524" layer="91"/>
-<label x="58.42" y="160.02" size="1.27" layer="95" xref="yes"/>
-</segment>
-</net>

Commit message: added milling layer for pannelization
Parts:
- added U$1: UMICH_SOLID_SMALL, logos:UMICH_SOLID_SMALL
